File: hardware/project-soic8-stemmaqt-mod.kicad_pcb (KiCad board)
At the start: 2 copper layers, 14.5 x 8.4 mm, 2 parts, among them J1 SM04B-SRSS-TB(LF)(SN), U1 24LC00

Commit message: Update version on board
Routing:
- net GND: track 4.36 -> 3.83 mm
Other:
- board text added: "v2.0.0"
- board text removed: "v1.0-3 -gf25257a"
